File: VDA.brd (EAGLE design)
At the start: 160 x 100 mm, 70 parts, among them J3 FTSH-107-01-L-DV-K-A, SW1 DSHP03TSGER, U1 SN74LVC1G175, U10 LP3966-3.3, U2 CP2102N-28, U3 STM32F373CBT6, U4 LP5907MFX-3.3/NOPB

Commit message: starting layout
Parts:
- removed C83, C84: 47u, Property-standar:A_3216
- removed R35: 270, Property-standar:R_0402
- removed U$7: USB-2.0, Connectors:USB-B
- removed U10: LP3966-3.3, property:TO-263
- added C24, C25, C28, C33, C34, C35, C36: 100n, Property-standar:C_0603
- added C26: 4u7, Property-standar:C_0603
- added C29, C30: 47n, Property-standar:C_0603
- added C31: 3.3u, Property-standar:C_0603
- added C32: 470n, Property-standar:C_0603
- added J1: USB-2.0, Connectors:USB-B
- added R10, R11, R9: 2k, Property-standar:R_0603
- added R12, R14: 30k, Property-standar:R_0603
- added R13, R8: 10k, Property-standar:R_0603
- added R22: 270, Property-standar:R_0402
- added R3, R4, R6, R7: 10M, Property-standar:R_0603
- added SJ1: (no value), property-pads:SJ_2
- added U5: ISO7721DR, property_digital:SO8
- added U6: LP5907MFX-3.3/NOPB, property-power:SOT23-5
- added U7: TL072, property:SOIC127P600X175-14N
- added U8: LM13700, property_analog:SO16
- D10: value YELLOW -> GREEN
- moved D11 324.7 mm to (-40.6, -429.3)
- moved R5 315.7 mm to (-43.2, -414.0)
- moved PS2 279.7 mm to (47.6, 72.4)
- moved PS1 261.4 mm to (47.6, 63.5)
- moved C1 240.7 mm to (15.2, 71.0), turned to 180 degrees
- moved R1 236.7 mm to (15.2, 72.9), turned to 180 degrees
- moved D4 155.9 mm to (28.6, 63.3)
- moved D3 152.6 mm to (31.1, 64.6), turned to 180 degrees
- moved R17 147.6 mm to (20.3, 51.3)
- moved D2 146.0 mm to (25.4, 64.0)
- moved R19 145.3 mm to (20.3, 55.1)
- moved R18 143.4 mm to (20.3, 53.2), turned to 180 degrees
- moved C6 133.8 mm to (22.9, 59.5), turned to 90 degrees
- moved C5 133.4 mm to (24.8, 59.5), turned to 90 degrees
- moved R16 133.2 mm to (52.1, 51.4), turned to 180 degrees
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Connections:
- net LED2 renamed LED_ACQ
- removed net FAULT_LED: R5.1
- removed net LED5: D11.K
- removed net N$24: U1.4, U3.44
- removed net N$29: D10.K, R5.2
- removed net N$36: D11.A, R35.2
- new net BOOT0: R22.1, U1.4, U3.44
- new net DAC_OUT: R14.1
- new net GND1: C30.P$2, R7.1, R9.2, U7.1
- new net LED_PWR: D10.K
- new net N$1: C26.P$1, C28.P$1, SJ16.2, TP3.TP, U6.5
- new net N$10: C32.P$1, R10.1, SJ1.NC, U7.14
- new net N$12: R13.1, U8.8
- new net N$13: R14.2, U8.1
- new net N$14: D10.A, R5.2
- new net N$15: D11.A, R22.2
- new net N$2: C29.P$1, R3.2, U7.3
- new net N$3: R3.1, R4.2
- new net N$4: C30.P$1, R6.2, R8.1, U7.2
- new net N$5: R6.1, R7.2
- new net N$6: R8.2, U$6.2
- new net N$7: C31.P$1, R10.2, R11.2, R9.1
- new net N$9: R12.1, U8.5, U8.7
- new net RXD: U2.25, U5.2
- new net TXD: U2.26, U5.3
- net +3V3: now also R5.1; no longer D10.A, R35.1
- net +5V: now also C25.P$1, C34.P$1, C36.P$1, U5.8, U6.1, U7.4, U8.11; no longer U10.2
- net -5V: now also C33.P$2, C35.P$2, R13.2, U7.11, U8.6
- net GND: now also C25.P$2, C26.P$2, C28.P$2, C29.P$2, C31.P$2, C33.P$1, C34.P$2, C35.P$1, C36.P$2, D11.K, R12.2, R4.1, U$6.1, U$6.3, U5.5, U6.2, U7.12; no longer C83.K, C84.K, U10.3, U10.6, U2.3, U2.EXP
- net GND-1: now also C24.P$2, J1.4, U2.3, U2.EXP, U5.4; no longer U$7.4
- net N$11: now also C32.P$2, R11.1, U7.13; no longer C83.A, C84.A, SJ16.2, TP3.TP, U10.4, U10.5
- net N$46: now also U6.3; no longer U10.1
- net SHIELD: now also J1.M1, J1.M2; no longer U$7.M1, U$7.M2
- net USB_DN: now also J1.2; no longer U$7.2
- net USB_DP: now also J1.3; no longer U$7.3
- net USB_RXD: now also U5.7; no longer U2.25
- net USB_TXD: now also U5.6; no longer U2.26
- net VUSB: now also C24.P$1, J1.1, U5.1; no longer U$7.1
Other:
- board size 160 x 100 mm -> 100 x 80 mm

Commit message: trabajando
Parts:
- moved C33 420.4 mm to (32.4, 30.5), turned to 270 degrees
- moved C34 417.3 mm to (32.4, 19.7), turned to 270 degrees
- moved R8 330.4 mm to (29.2, 14.6), turned to 270 degrees
- moved C36 328.5 mm to (-17.1, -78.7)
- moved C30 328.4 mm to (28.6, 20.3), turned to 180 degrees
- moved D11 321.5 mm to (75.6, -129.5)
- moved R22 321.5 mm to (73.0, -121.9)
- moved R5 321.5 mm to (73.0, -114.3)
- moved C35 320.3 mm to (-28.6, -78.7)
- moved R7 318.5 mm to (25.4, 18.4)
- moved R6 311.6 mm to (28.6, 18.4)
- moved R14 303.9 mm to (-29.2, -72.4)
- moved C29 303.7 mm to (32.4, 17.1)
- moved R4 293.9 mm to (33.0, 14.6), turned to 270 degrees
- moved C21 293.6 mm to (41.3, 74.9)
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Connections:
- new net N$6: SJ1.COM, U$6.1, U$6.3
- new net NRST: C13.P$2, R28.1, S3.P$1, S3.P$2, U3.7
- net GND: now also SJ1.NO; no longer U$6.1, U$6.3
- net N$10: no longer SJ1.NC
- net N$2: now also SJ1.NC
- net NRST_2: no longer C13.P$2, R28.1, S3.P$1, S3.P$2, U3.7
Other:
- outline, holes or cut-outs redrawn

Commit message: inicio layout
Parts:
- added R23: 100, Property-standar:R_0603
- added R27: 10k, Property-standar:R_0603
- added SHIELD: MS384, shields:MS384
- R8: value 10k -> 100
- moved C3 181.2 mm to (88.9, 45.1)
- moved R2 178.6 mm to (88.9, 46.4), turned to 180 degrees
- moved C2 176.1 mm to (88.9, 47.6)
- moved D11 172.0 mm to (88.9, 41.9)
- moved U1 168.0 mm to (84.8, 45.5)
- moved R22 165.9 mm to (88.9, 43.2)
- moved SJ4 109.9 mm to (91.4, 54.0), turned to 180 degrees
- moved C15 64.6 mm to (67.3, 66.0), turned to 180 degrees
- moved C16 62.5 mm to (67.3, 64.8), turned to 180 degrees
- moved C14 61.3 mm to (69.8, 58.4), turned to 180 degrees
- moved C17 57.7 mm to (69.8, 59.7), turned to 180 degrees
- moved R5 56.6 mm to (33.7, -73.7)
- moved C18 54.7 mm to (74.3, 71.1)
- moved R21 47.7 mm to (89.5, 67.3), turned to 0 degrees
- moved C11 38.5 mm to (83.2, 67.9), turned to 0 degrees
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Connections:
- net +3V3A1 renamed FF_CLR
- net JCLK_2 renamed JCLK
- net JRCLK_2 renamed JRCLK
- net JTDI_2 renamed JTDI
- net JTDO_2 renamed JTDO
- net JTMS_2 renamed JTMS
- removed net NRST_2: J3.12
- removed net SAMPLING_ZCD: U3.32
- removed net TRIGGER_ZCD: U3.29
- new net FF_CLK: U1.1, U3.45
- new net FF_D: U1.3, U3.46
- new net N$17: R23.2, SJ1.NC
- new net N$18: R22.1, U1.4
- net BOOT0: now also R27.1; no longer R22.1, U1.4
- net GND: now also R27.2, SHIELD.P$1, SHIELD.P$2
- net N$2: now also R23.1; no longer SJ1.NC
- net NRST: now also J3.12
Routing:
- net NRST: track 0.00 -> 37.5 mm, vias 0 -> 2
- net GND-1: track 0.00 -> 31.0 mm, vias 0 -> 13
- net VUSB: track 0.00 -> 30.0 mm, vias 0 -> 5
- net USART_TX: track 0.00 -> 25.3 mm, vias 0 -> 2
- net USART_RX: track 0.00 -> 25.2 mm, vias 0 -> 2
- net GND: track 0.00 -> 22.0 mm, vias 0 -> 14
- net VDD_BRIDGE: track 0.00 -> 19.3 mm, vias 0 -> 2
- net SHIELD: track 0.00 -> 19.3 mm
- net ON_MODE: track 0.00 -> 17.2 mm
- net USB_DP: track 0.00 -> 16.7 mm
- net RS_MODE: track 0.00 -> 16.7 mm
- net JCLK: track 0.00 -> 16.6 mm, vias 0 -> 2
- net SP_MODE: track 0.00 -> 16.6 mm
- net USB_DN: track 0.00 -> 13.9 mm
- net JRCLK: track 0.00 -> 13.8 mm, vias 0 -> 2
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- added copper zone on layer 1, net +3V3
- added copper zone on layer 1, net +3V3A
- added copper zone on layer 2, net GND
- added copper zone on layer 2, net GND-1
- added copper zone on layer 15, net VUSB
Other:
- board size 100 x 80 mm -> 100 x 90 mm

Commit message: trabajando en el layout
Parts:
- added C37, C38: 22u, Property-standar:CAPAE660X590N
- added C39: 4u7, Property-standar:C_0603
- added C40: 100n, Property-standar:C_0603
- added C41: 10u, Property-standar:C_0603
- added R29: (no value), Property-standar:POT-09VR1M
- added SJ2: (no value), jumper:SJ
- added TP1, TP2, TP4: HOLE_0.8MM, property-connectors:HOLE_0.8MM
- added U9: REF3433IDBVR, Power-Supply:SOT23-6
- C22, C23: value 10u -> 100n
- SJ1: device property-pads:SJ_2 -> jumper:SJ_2
- TP3: value TPB1,27 -> HOLE_0.8MM; device testpad:B1,27 -> property-connectors:HOLE_0.8MM
- moved C26 194.4 mm to (80.6, 81.3)
- moved C28 192.6 mm to (80.6, 83.2)
- moved U6 183.1 mm to (80.6, 78.1)
- moved TP3 177.1 mm to (80.0, 85.7)
- moved SJ16 172.1 mm to (77.5, 81.9), turned to 90 degrees
- moved C79 161.1 mm to (84.5, 78.7)
- moved R111 160.8 mm to (84.5, 76.8)
- moved C80 149.2 mm to (80.6, 74.3)
- moved C81 145.8 mm to (80.6, 71.8)
- moved C20 145.8 mm to (95.2, 46.4)
- moved SJ6 137.8 mm to (92.1, 45.1), turned to 90 degrees
- moved C27 136.7 mm to (95.2, 38.1)
- moved D5 132.3 mm to (92.1, 40.6), turned to 270 degrees
- moved C19 131.1 mm to (95.2, 44.5)
- moved U4 122.2 mm to (95.2, 41.3)
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Connections:
- new net MANUAL_GAIN: R29.P$3
- new net N$19: C39.P$1, C40.P$1, SJ2.2, U9.5, U9.6
- net +3V3A: now also R29.P$1, SJ2.1
- net +5V: now also C37.+, C41.P$1, TP1.1, U9.3, U9.4
- net -5V: now also C38.-, TP4.1
- net FF_CLK: now also U3.46; no longer U3.45
- net FF_D: now also U3.45; no longer U3.46
- net GND: now also C37.-, C38.+, C39.P$2, C40.P$2, C41.P$2, R29.P$2, SJ1.3, TP2.1, U9.1, U9.2; no longer SJ1.NO
- net N$1: now also TP3.1; no longer TP3.TP
- net N$17: now also SJ1.1; no longer SJ1.NC
- net N$6: now also SJ1.2; no longer SJ1.COM
Routing:
- net -5V: track 0.00 -> 29.4 mm
- net USART_TX: track 25.3 -> 50.8 mm
- net +5V: track 2.95 -> 27.1 mm
- net USART_RX: track 25.2 -> 41.7 mm
- net NRST: track 37.5 -> 22.7 mm
- net FF_D: track 0.00 -> 13.1 mm
- net FF_CLK: track 0.00 -> 10.4 mm
- net JTDI: track 10.2 -> 18.3 mm
- net JCLK: track 16.6 -> 23.8 mm, vias 2 -> 3
- net JTDO: track 10.3 -> 17.4 mm, vias 0 -> 2
- net GND: track 22.0 -> 26.3 mm, vias 14 -> 19
- net FF_CLR: track 0.00 -> 3.82 mm
- net +3V3: track 12.9 -> 16.5 mm, vias 5 -> 7
- net JTMS: track 13.4 -> 16.9 mm
- net MCU_RX: track 0.00 -> 2.90 mm
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- added copper zone on layer 1, net GND
