File: VDA.sch (EAGLE design)
At the start: 70 parts, among them J3 FTSH-107-01-L-DV-K-A, SW1 DSHP03TSGER, U1 SN74LVC1G175, U10 LP3966-3.3, U2 CP2102N-28, U3 STM32F373CBT6, U4 LP5907MFX-3.3/NOPB

Commit message: starting layout
Parts:
- removed C83, C84: 47u, Property-standar:C-TANTALUM_A_3216
- removed R35: 270, Property-standar:R_0402
- removed U10: LP3966-3.3, property:LP3966
- added C24, C25, C28, C33, C34, C35, C36: 100n, Property-standar:C_0603
- added C26: 4u7, Property-standar:C_0603
- added C29, C30: 47n, Property-standar:C_0603
- added C31: 3.3u, Property-standar:C_0603
- added C32: 470n, Property-standar:C_0603
- added R10, R11, R9: 2k, Property-standar:R_0603
- added R12, R14: 30k, Property-standar:R_0603
- added R13, R8: 10k, Property-standar:R_0603
- added R22: 270, Property-standar:R_0402
- added R3, R4, R6, R7: 10M, Property-standar:R_0603
- added SJ1: (no value), property-pads:SJ-PS
- added U5: ISO7721DR, property_digital:ISO7721DR
- added U6: LP5907MFX-3.3/NOPB, property-power:LDO1SOT23-5_1
- added U7: TL072, property:LM324BD
- added U8: LM13700, property_analog:LM13700
- D10: value YELLOW -> GREEN
- renumbered U$7 to J1
Connections:
- net LED2 renamed LED_ACQ
- removed net FAULT_LED: R5.1
- removed net LED5: D11.K
- removed net N$24: U1.Q, U3.BOOT0
- removed net N$29: D10.K, R5.2
- removed net N$36: D11.A, R35.2
- new net BOOT0: R22.1, U1.Q, U3.BOOT0
- new net DAC_OUT: R14.1
- new net GND1: C30.2, R7.1, R9.2, U71.OUT
- new net LED_PWR: D10.K
- new net N$1: C26.1, C28.1, SJ16.2, TP3.TP, U6.OUT
- new net N$10: C32.1, R10.1, SJ1.NC, U74.OUT
- new net N$12: R13.1, U8_1.E
- new net N$13: R14.2, U8_1.AMP_BIAS
- new net N$14: D10.A, R5.2
- new net N$15: D11.A, R22.2
- new net N$2: C29.1, R3.2, U71.+IN
- new net N$3: R3.1, R4.2
- new net N$4: C30.1, R6.2, R8.1, U71.-IN
- new net N$5: R6.1, R7.2
- new net N$6: R8.2, U$6.TIP
- new net N$7: C31.1, R10.2, R11.2, R9.1
- new net N$9: R12.1, U8_1.B, U8_1.OUT
- new net RXD: U2.RXD, U5.OUT_A
- new net TXD: U2.TXD, U5.IN_B
- net +3V3: now also R5.1; no longer D10.A, R35.1
- net +5V: now also C25.1, C34.1, C36.1, U5.VCC2, U6.IN, U7P.V+, U8_P.V+; no longer U10.VIN
- net -5V: now also C33.2, C35.2, R13.2, U7P.V-, U8_P.V-
- net GND: now also C25.2, C26.2, C28.2, C29.2, C31.2, C33.1, C34.2, C35.1, C36.2, D11.K, R12.2, R4.1, U$6.RING, U$6.SLEEVE, U5.GND2, U6.GND, U74.+IN; no longer C83.-, C84.-, U10.GND, U2.GND, U2.GND@EXP
- net GND-1: now also C24.2, U2.GND, U2.GND@EXP, U5.GND1
- net N$11: now also C32.2, R11.1, U74.-IN; no longer C83.+, C84.+, SJ16.2, TP3.TP, U10.SNS/!ERR!, U10.VOUT
- net N$46: now also U6.EN; no longer U10.!SD!
- net USB_RXD: now also U5.INA_A; no longer U2.RXD
- net USB_TXD: now also U5.OUT_B; no longer U2.TXD
- net VUSB: now also C24.1, U5.VCC1
Other:
- note added: "ACQ LED"
- note added: "CLoad=(C1*C2/(C1+C2))+Cstray"
- note added: "CONECTAR FF"
- note added: "ISOLATED POWER SUPPLY"
- note added: "LM13700 Power"
- note added: "Power LED"
- note added: "Referencia de voltaje"
- note added: "TL072 Power"
- note added: "USB-TTL MCU"
- note added: "VERIFICAR QUE TX-RX ESTEN CORRECTOS VERIFICAR CORRECTA ORIENTACION DE IN-OUT AISLADOR"
- note removed: "ETH1"
- note removed: "ETH1 LED"
- note removed: "ETH2"
- note removed: "ETH2 LED"
- note removed: "Fault LED"
- note removed: "USB-TTL MCU 2"
- moved on the sheet: C10, C19, C2, C20, C21, C22, C23, C27, C3, C4, C79, C80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

Commit message: trabajando
Connections:
- new net N$6: SJ1.COM, U$6.RING, U$6.SLEEVE
- new net NRST: C13.2, R28.1, S3.P$1, U3.NRST
- net GND: now also SJ1.NO; no longer U$6.RING, U$6.SLEEVE
- net N$10: no longer SJ1.NC
- net N$2: now also SJ1.NC
- net NRST_2: no longer C13.2, R28.1, S3.P$1, U3.NRST
Other:
- note added: "Revisar: https://www.ti.com/litv/pdf/slyt369"
- moved on the sheet: SJ1, U$6

Commit message: inicio layout
Parts:
- added R23: 100, Property-standar:R_0603
- added R27: 10k, Property-standar:R_0603
- added SHIELD: MS384, shields:MS384
- R8: value 10k -> 100
Connections:
- net +3V3A1 renamed FF_CLR
- net JCLK_2 renamed JCLK
- net JRCLK_2 renamed JRCLK
- net JTDI_2 renamed JTDI
- net JTDO_2 renamed JTDO
- net JTMS_2 renamed JTMS
- removed net NRST_2: J3.12
- removed net SAMPLING_ZCD: U3.PA11
- removed net TRIGGER_ZCD: U3.PA8
- new net FF_CLK: U1.CLK, U3.PB8
- new net FF_D: U1.D, U3.PB9
- new net N$17: R23.2, SJ1.NC
- new net N$18: R22.1, U1.Q
- net BOOT0: now also R27.1; no longer R22.1, U1.Q
- net GND: now also R27.2, SHIELD.1
- net N$2: now also R23.1; no longer SJ1.NC
- net NRST: now also J3.12
Other:
- note added: "BOOT0 managment circuit"
- note added: "Differential Charge-Amp"
- note added: "MS384-10F MS384-10C"
- note removed: "CONECTAR FF"
- note removed: "EXTI11"
- note removed: "TIM5_CH1"
- moved on the sheet: C2, C3, D11, R2, R20, R21, R22, R24, R25, R26, R8, SJ1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

Commit message: trabajando en el layout
Parts:
- added C37, C38: 22u, Property-standar:C-ELECT-6.3X5.4
- added C39: 4u7, Property-standar:C_0603
- added C40: 100n, Property-standar:C_0603
- added C41: 10u, Property-standar:C_0603
- added R29: (no value), Property-standar:R-VARIABLE09VR1B
- added SJ2: (no value), jumper:SJ
- added TP1, TP2, TP4: HOLE_0.8MM, property-connectors:HOLE_0.8MM
- added U9: REF3433IDBVR, Power-Supply:REF3433IDBVR
- C22, C23: value 10u -> 100n; V 16V -> (none)
- SJ1: device property-pads:SJ-PS -> jumper:SJ2W
- TP3: value TPB1,27 -> HOLE_0.8MM; device testpad:TPB1,27 -> property-connectors:HOLE_0.8MM
Connections:
- new net MANUAL_GAIN: R29.C
- new net N$19: C39.1, C40.1, SJ2.2, U9.OUT_F, U9.OUT_S
- net +3V3A: now also R29.1, SJ2.1
- net +5V: now also C37.+, C41.1, TP1.P, U9.EN, U9.IN
- net -5V: now also C38.-, TP4.P
- net FF_CLK: now also U3.PB9; no longer U3.PB8
- net FF_D: now also U3.PB8; no longer U3.PB9
- net GND: now also C37.-, C38.+, C39.2, C40.2, C41.2, R29.2, SJ1.3, TP2.P, U9.GND_F, U9.GND_S; no longer SJ1.NO
- net N$1: now also TP3.P; no longer TP3.TP
- net N$17: now also SJ1.1; no longer SJ1.NC
- net N$6: now also SJ1.2; no longer SJ1.COM
Other:
- note added: "Voltage Reference"
- note removed: "Referencia de voltaje"
- moved on the sheet: C19, C20, C22, C23, SJ6
