File: Panel Frontal/Panel Frontal/Panel Frontal.sch (EAGLE design)
At the start: 16 parts, among them J1 F0504-H-05-10G-R, Q1 BSS138, Q2 BSS138, Q3 BSS138

Commit message: layout avanzado
Other:
- note added: "ACQ LED"
- note added: "PROG LED"
- note added: "Power LED"
Changed lines of the file:
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@@
 <schematic xreflabel="%F%N/%S.%C%R" xrefpart="/%S.%C%R">
 <attributes>
+<attribute name="VERSION" value="1.0"/>
 </attributes>
 <variantdefs>
@@
 <part name="+3V3" library="USBC_LBRY" deviceset="+3V3" device=""/>
 <part name="R3" library="Property-standar" library_urn="urn:adsk.eagle:library:20126172" deviceset="R" device="_0603" package3d_urn="urn:adsk.eagle:package:39983384/2" value="100R"/>
-<part name="FRAME1" library="Frames" library_urn="urn:adsk.eagle:library:46102009" deviceset="FRAMES" device=""/>
+<part name="FRAME1" library="Frames" library_urn="urn:adsk.eagle:library:46102009" deviceset="FRAMES" device="">
+<attribute name="VERSION" value=""/>
+</part>
 <part name="+3V4" library="USBC_LBRY" deviceset="+3V3" device=""/>
 <part name="D2" library="property_LED" library_urn="urn:adsk.eagle:library:46147719" deviceset="LED-REVERSE_MOUNT" device="" package3d_urn="urn:adsk.eagle:package:46147722/4"/>
@@
 <description>Panel Frontal</description>
 <plain>
-<text x="58.42" y="48.26" size="1.778" layer="97">VLRK31Q1R2-GS08</text>
+<text x="48.26" y="63.5" size="1.778" layer="97">VLRK31Q1R2-GS08</text>
+<text x="183.388" y="167.64" size="3.81" layer="97">Power LED</text>
+<text x="150.368" y="167.64" size="3.81" layer="97">ACQ LED</text>
+<text x="112.268" y="167.64" size="3.81" layer="97">PROG LED</text>
 </plain>
 <instances>
@@
 <attribute name="SHEET_HEADLINE" x="185.42" y="12.7" size="3.81" layer="97"/>
 <attribute name="LAST_DATE_TIME" x="195.58" y="1.27" size="2.54" layer="97"/>
+<attribute name="VERSION" x="251.46" y="1.27" size="2.54" layer="97"/>
 </instance>
 <instance part="+3V4" gate="G$1" x="63.5" y="86.36" smashed="yes" rot="MR0">
