File: Panel Posterior/Panel Posterior/Panel Posterior.brd (EAGLE design)
At the start: 130 x 50 mm, 1 part

Commit message: layout avanzado
Changed lines of the file:
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@@
 </layers>
 <board>
-<fusionsync huburn="a.cGVyc29uYWw6dWUyZjQ5ODk2" projecturn="a.cGVyc29uYWw6dWUyZjQ5ODk2IzIwMjQxMjMwODUxNjE5OTA2" f3durn="urn:adsk.wipprod:dm.lineage:EEgtof-oSiOk8acphO_9ag" pcbguid="" lastpulledtime="" lastsyncedchangeguid="" latestrevisionid="6b66e87f-6855-4784-81f6-0fe28c529530" lastsyncedrevisionid="6b66e87f-6855-4784-81f6-0fe28c529530" lastboardhashguid="3af134c1-92bf-fac7-ff68-25addc0c63ec" lastpushedtime="2025-01-06T01:32:56Z" linktopcb3d="true"/>
+<fusionsync huburn="a.cGVyc29uYWw6dWUyZjQ5ODk2" projecturn="a.cGVyc29uYWw6dWUyZjQ5ODk2IzIwMjQxMjMwODUxNjE5OTA2" f3durn="urn:adsk.wipprod:dm.lineage:EEgtof-oSiOk8acphO_9ag" pcbguid="" lastpulledtime="" lastsyncedchangeguid="" latestrevisionid="8b1f6ea9-1bfc-438c-b0c2-f471490725e8" lastsyncedrevisionid="8b1f6ea9-1bfc-438c-b0c2-f471490725e8" lastboardhashguid="3af134c1-92bf-fac7-ff68-25addc0c63ec" lastpushedtime="2025-01-06T19:19:04Z" linktopcb3d="true"/>
 <plain>
 <wire x1="0" y1="0" x2="130" y2="0" width="0" layer="20"/>
@@
 </autorouter>
 <elements>
-<element name="U$2" library="Frames" library_urn="urn:adsk.eagle:library:46102009" package="LOGO_VDA-3CM" package3d_urn="urn:adsk.eagle:package:46150161/1" value="LOGO_VDA-3CM" x="23" y="10" smashed="yes"/>
+<element name="U$2" library="Frames" library_urn="urn:adsk.eagle:library:46102009" package="LOGO_VDA-3CM" package3d_urn="urn:adsk.eagle:package:46150161/3" value="LOGO_VDA-3CM" x="23" y="10" smashed="yes"/>
 </elements>
 <signals>
