File: Panelizado_frentes/Panelizado_frentes.sch (EAGLE design)
At the start: 17 parts, among them J2 F0504-H-05-10G-R, Q4 BSS138, Q5 BSS138, Q6 BSS138

Commit message: BOM del adquisidor listo
Parts:
- renumbered J2 to J1, Q4 to Q1, Q5 to Q2, Q6 to Q3, R10 to R2, R11 to R1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
