File: Adquisidor en español/VDA spanish.sch (EAGLE design)
At the start: 137 parts, among them J1 USB-2.0, J2 CONVERT-1X4-2.54MM-MALE_HOLES, J3 FTSH-107-01-L-DV-K-A, J4 STEREO-JACK, J5 F0504-H-05-10G-R, J6 CONVERT-2X7-2.54MM-FEMALE, Q1 BC856, Q2 BC856, SW1 DSHP03TSGER, U1 CP2102N-28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

Commit message: Archivos mas ordenados
Other:
- note added: "Amplificador Controlado por Tensión"
- note added: "Amplificador de Carga Diferencial"
- note added: "Amplificador y Offset"
- note added: "CIRCUITO DE CONTROL DE BOOT0"
- note added: "CONVERSOR USB-UART"
- note added: "Conector de Expansión"
- note added: "Conector para panel Frontal"
- note added: "Conversor Corriente - Tensión"
- note added: "Conversor Tensión - Corriente"
- note added: "FUENTE DE ALIMENTACIÓN AISLADA"
- note added: "FUENTE DE ALIMENTACIÓN PARA MCU (DOMINIO ANALÓGICO)"
- note added: "FUENTE DE ALIMENTACIÓN PARA MCU (DOMINIO DIGITAL)"
- note added: "No usado LM13700 1/2"
- note added: "UART AISLADA"
- note removed: "Amplifier and Offset"
- note removed: "BOOT0 managment circuit"
- note removed: "Current to Voltage"
- note removed: "Differential Charge-Amp"
- note removed: "Expansion Connector"
- note removed: "Front Panel Connector"
- note removed: "ISOLATED POWER SUPPLY"
- note removed: "ISOLATED UART"
- note removed: "POWER SUPPLY FOR MCU (ANALOG DOMAIN)"
- note removed: "POWER SUPPLY FOR MCU (DIGITAL DOMAIN)"
- note removed: "USB-TTL MCU"
- note removed: "Unused LM13700 1/2"
- note removed: "Voltage - Current Converter"
- note removed: "Voltage Controlled Amplifier"
- moved on the sheet: C22, C23, C24, C25, C26, C27, C28, C29, C30, C31, C32, C33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
